File: zz_RJ45_to_zh.kicad_pcb (KiCad board)
At the start: 2 copper layers, 31 x 55 mm, 10 parts, among them J1 RJ45-B-1_1, J2 S6B-ZR-SM2-TF__LF__SN_

Commit message: modify
Parts:
- removed R1, R2, R3, R4, R5, R6: 51, Resistor_SMD:R_0603_1608Metric
- removed R7: 75, Resistor_SMD:R_0603_1608Metric
- added C2: 0.1uF, Capacitor_SMD:C_0603_1608Metric, F.Cu at (197.6, 105.0)
- added C4: CL31B102KJHNNNE, SamaSys_Parts:CAPC3216X180N, F.Cu at (199.8, 104.4)
- C1: value 1000pF -> 0.1uF
- J1: value RJ45-B-1_1 -> Conn_02x03_Top_Bottom; footprint SamaSys_Parts:RJ45B11 -> Connector_PinSocket_2.54mm:PinSocket_2x03_P2.54mm_Horizontal
- J2: value S6B-ZR-SM2-TF__LF__SN_ -> RJMG1S8008101BR; footprint SamaSys_Parts:S6BZRSM2TFLFSN -> me:AMPHENOL_RJMG1S8008101BR
- moved J2 31.0 mm to (195.4, 118.8), turned to 0 degrees
- moved J1 13.9 mm to (178.4, 117.0), turned to 90 degrees
- moved C1 4.83 mm to (195.2, 105.0), turned to 90 degrees
Connections:
- C1 pad 1: Net-(C1-Pad1) -> Net-(J2-TCT2)
- J1 pad 1: Net-(J1-Pad1) -> ETH_TX1P
- J1 pad 2: Net-(J1-Pad2) -> ETH_TX1N
- J1 pad 3: Net-(J1-Pad3) -> ETH_RX1P
- J1 pad 4: Net-(J1-Pad4) -> ETH_RX1N
- J1 pad 5: Net-(J1-Pad5) -> GND
- J1 pad 6: Net-(J1-Pad6) -> GND
- J2 pad 1: Net-(J1-Pad6) -> ETH_TX1P
- J2 pad 2: Net-(J1-Pad3) -> ETH_TX1N
- J2 pad 3: Net-(J1-Pad2) -> Net-(J2-TCT1)
- J2 pad 4: Net-(J1-Pad1) -> unconnected-(J2-NA1-Pad4)
- J2 pad 5: /CMT -> unconnected-(J2-NA2-Pad5)
- J2 pad 6: GND -> Net-(J2-TCT2)
Routing:
- net Net-(J1-Pad6): track 43.6 -> 0.00 mm, vias 1 -> 0
- net Net-(J1-Pad2): track 36.8 -> 0.00 mm
- net Net-(J1-Pad1): track 36.5 -> 0.00 mm, vias 2 -> 0
- net Net-(J1-Pad3): track 34.7 -> 0.00 mm, vias 1 -> 0
- net GNDS: track 0.00 -> 34.2 mm, vias 0 -> 8
- net ETH_RX1N: track 0.00 -> 26.1 mm
- net /CMT: track 22.6 -> 0.00 mm
- net ETH_TX1N: track 0.00 -> 21.8 mm
- net GND: track 36.0 -> 56.5 mm, vias 44 -> 37
- net ETH_RX1P: track 0.00 -> 20.4 mm
- net ETH_TX1P: track 0.00 -> 16.3 mm
- net Net-(J1-Pad8): track 13.1 -> 0.00 mm
- net Net-(J1-Pad5): track 11.7 -> 0.00 mm
- net Net-(J1-Pad4): track 11.1 -> 0.00 mm
- net Net-(J2-TCT1): track 0.00 -> 10.6 mm
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- added copper zone on B.Cu, net GNDS
- added copper zone on F.Cu, net GNDS
Other:
- board text added: "TXP RXP GND TXN RXN GND"
