File: zz_RJ45_to_zh.kicad_sch (KiCad schematic)
At the start: 10 parts, among them J1 RJ45-B-1_1, J2 S6B-ZR-SM2-TF__LF__SN_

Commit message: modify
Parts:
- removed C1: 1000pF, Capacitor_SMD:C_0603_1608Metric, symbol Device:C_Small_US
- removed J1: RJ45-B-1_1, SamaSys_Parts:RJ45B11, symbol SamacSys_Parts:RJ45-B-1_1
- removed J2: S6B-ZR-SM2-TF__LF__SN_, SamaSys_Parts:S6BZRSM2TFLFSN, symbol SamacSys_Parts:S6B-ZR-SM2-TF__LF__SN_
- removed R1, R2, R3, R4, R5, R6: 51, Resistor_SMD:R_0603_1608Metric, symbol Device:R
- removed R7: 75, Resistor_SMD:R_0603_1608Metric, symbol Device:R
- added C1, C2: 0.1uF, Capacitor_SMD:C_0603_1608Metric, symbol Device:C
- added C4: CL31B102KJHNNNE, SamaSys_Parts:CAPC3216X180N, symbol SamacSys_Parts:CL31B102KJHNNNE
- added J1: Conn_02x03_Top_Bottom, Connector_PinSocket_2.54mm:PinSocket_2x03_P2.54mm_Horizontal, symbol Connector_Generic:Conn_02x03_Top_Bottom
- added J2: RJMG1S8008101BR, me:AMPHENOL_RJMG1S8008101BR, symbol me:RJMG1S8008101BR
Connections:
- net GND: now also C1.2, C2.2, C4.1, J1.5 (Pin_5), J1.6 (Pin_6)
- new net: C2.1, J2.3 (TCT1)
- new net: C1.1, J2.6 (TCT2)
- new net ETH_RX1N: J1.4 (Pin_4), J2.8 (RD-)
- new net ETH_RX1P: J1.3 (Pin_3), J2.7 (RD+)
- new net ETH_TX1N: J1.2 (Pin_2), J2.2 (TD-)
- new net ETH_TX1P: J1.1 (Pin_1), J2.1 (TD+)
- new net GNDS: C4.2, J2.S1 (SHIELD), J2.S2 (SHIELD__1)
- no-connect marks 2 -> 0
Other:
- note added: "6:GND 5:CMT 4:RX1- 3:RX1+ 2:TX1- 1:TX1+"
- note added: "H1102 回路図"
- note added: "Pulse Transmitterを含むRJ45 connector"
- note added: "chassis GND"
- note added: "理想的にはnetwork機器側に置くが、 TCMT,RCMT,GNDをpinにだすと 信号線が増えてしまうので また、このCは共有できない"
- note removed: "4:TX1+ 3:TX1- 2:RX1+ 1:RX1-"
- note removed: "8: 7: 6:RX1- 5: 4: 3:RX1+ 2:TX1- 1:TX1+"
